Commit message: fix: variable in car.xacro

File: urdf/car.xacro (robot description, xacro)
@@ -4,20 +4,21 @@
     <xacro:property name="body_link_y_dim" value="0.6"/>
     <xacro:property name="body_link_z_dim" value="0.3"/>
-    <xacro:property name="wheel_link_radius" value="0.1"/>
-    <xacro:property name="wheel_link_length" value="0.2"/>
+    <xacro:property name="wheel_link_radius" value="0.15"/>
+    <xacro:property name="wheel_link_length" value="0.1"/>
     <xacro:property name="wheel_link_z_location" value="-0.1"/>
     <xacro:property name="body_density" value="2710.0"/>
-    <xacro:property name="wheel_dentisy" value="2710.0"/>
+    <xacro:property name="wheel_desity" value="2710.0"/>
     <xacro:property name="pi_const" value="3.14159265"/>
     <xacro:property name="body_mass" value="${body_density*body_link_x_dim*body_link_y_dim*body_link_z_dim}"/>
     <xacro:property name="wheel_mass"
-    value="${wheel_dentisy*wheel_link_length*wheel_link_radius*wheel_link_radius*pi_const}"/>
+        value="${wheel_desity*wheel_link_length*wheel_link_radius*wheel_link_radius*pi_const}"/>
     <xacro:property name="Iz_wheel" value="${0.5*wheel_mass*wheel_link_radius*wheel_link_radius}"/>
-    <xacro:property name="I_wheel" value="${(1.0/12.0)/wheel_mass*(3.0*wheel_link_radius*wheel_link_radius+wheel_link_length*wheel_link_length)}"/>
+    <xacro:property name="I_wheel"
+        value="${(1.0/12.0)*wheel_mass*(3.0*wheel_link_radius*wheel_link_radius+wheel_link_length*wheel_link_length)}"/>
     <xacro:macro name="inertia_wheel">
         <inertial>
-            <origin rpy="0 0 0" xyz="0 0 0"/>
+            <origin rpy="0.0 0.0 0.0" xyz="0.0 0.0 0.0"/>
             <mass value="${wheel_mass}"/>
-            <inertia ixx="${I_wheel}" ixy="0.0" ixz="${.00}" iyy="${I_wheel}" izz="${Iz_wheel}" iyz="0"/>
+            <inertia ixx="${I_wheel}" ixy="0.0" ixz="0.0" iyy="${I_wheel}" izz="${Iz_wheel}" iyz="0.0"/>
         </inertial>
     </xacro:macro>
@@ -41,10 +42,11 @@
             <origin xyz="0.0 0.0 0.0" rpy="0.0 0.0 0.0"/>
             <mass value="${body_mass}"/>
-            <inertia    ixx="${(1/12)/body_mass*(body_link_y_dim*body_link_y_dim+body_link_z_dim*body_link_z_dim)}"
-                        ixy="0.0"
-                        ixz="0.0"
-                        iyy="${(1/12)/body_mass*(body_link_x_dim*body_link_x_dim+body_link_z_dim*body_link_z_dim)}"
-                        iyz="0.0"
-                        izz="${(1/12)/body_mass*(body_link_y_dim*body_link_y_dim+body_link_x_dim*body_link_x_dim)}"/>
+            <inertia
+                ixx="${(1/12)*body_mass*(body_link_y_dim*body_link_y_dim+body_link_z_dim*body_link_z_dim)}"
+                ixy="0"
+                ixz="0"
+                iyy="${(1/12)*body_mass*(body_link_x_dim*body_link_x_dim+body_link_z_dim*body_link_z_dim)}"
+                iyz="0"
+                izz="${(1/12)*body_mass*(body_link_y_dim*body_link_y_dim+body_link_x_dim*body_link_x_dim)}"/>
         </inertial>
         <collision>
@@ -60,13 +62,13 @@
         <parent link="body_link"/>
         <child link="wheel1_link"/>
-        <origin xyz="${-body_link_x_dim/2+1/2*wheel_link_radius} ${-body_link_y_dim/2 - wheel_link_length/2} ${wheel_link_z_location}"
+        <origin xyz="${-body_link_x_dim/2+1.2*wheel_link_radius} ${-body_link_y_dim/2 - wheel_link_length/2} ${wheel_link_z_location}"
                 rpy="0.0 0.0 0.0"/>
-        <axis xyz="0.0 1.0 0.0"/>
+        <axis xyz="0 1 0"/>
         <limit effort="1000.0" velocity="1000.0"/>
-        <dynamics damping="1" friction="1"/>
+        <dynamics damping="1.0" friction="1.0"/>
     </joint>
     <link name="wheel1_link">
         <visual>
-            <origin xyz="0 0 0" rpy="1.570795 0 0"/>
+            <origin xyz="0.0 0.0 0.0" rpy="1.570795 0 0"/>
             <geometry>
                 <cylinder radius="${wheel_link_radius}" length="${wheel_link_length}"/>
@@ -74,5 +76,5 @@
         </visual>
         <collision>
-            <origin xyz="0 0 0" rpy="1.570795 0 0"/>
+            <origin xyz="0.0 0.0 0.0" rpy="1.570795 0 0"/>
             <geometry>
                 <cylinder radius="${wheel_link_radius}" length="${wheel_link_length}"/>
@@ -86,13 +88,13 @@
         <parent link="body_link"/>
         <child link="wheel2_link"/>
-        <origin xyz="${-body_link_x_dim/2 + wheel_link_radius/2} ${body_link_y_dim/2 + wheel_link_length/2} ${wheel_link_z_location}"
+        <origin xyz="${-body_link_x_dim/2 + 1.2*wheel_link_radius} ${body_link_y_dim/2 + wheel_link_length/2} ${wheel_link_z_location}"
                 rpy="0.0 0.0 0.0"/>
         <axis xyz="0 1 0"/>
         <limit effort="1000.0" velocity="1000.0"/>
-        <dynamics damping="1" friction="1"/>
+        <dynamics damping="1.0" friction="1.0"/>
     </joint>
     <link name="wheel2_link">
         <visual>
-            <origin xyz="0 0 0" rpy="1.570795 0 0"/>
+            <origin xyz="0.0 0.0 0.0" rpy="1.570795 0 0"/>
             <geometry>
                 <cylinder radius="${wheel_link_radius}" length="${wheel_link_length}"/>
@@ -100,5 +102,5 @@
         </visual>
         <collision>
-            <origin xyz="0 0 0" rpy="1.570795 0 0"/>
+            <origin xyz="0.0 0.0 0.0" rpy="1.570795 0 0"/>
             <geometry>
                 <cylinder radius="${wheel_link_radius}" length="${wheel_link_length}"/>
@@ -112,13 +114,13 @@
         <parent link="body_link"/>
         <child link="wheel3_link"/>
-        <origin xyz="${body_link_x_dim/2 - wheel_link_radius/2} ${-body_link_y_dim/2 - wheel_link_length/2} ${wheel_link_z_location}"
+        <origin xyz="${body_link_x_dim/2 - 1.2*wheel_link_radius} ${-body_link_y_dim/2 - wheel_link_length/2} ${wheel_link_z_location}"
                 rpy="0.0 0.0 0.0"/>
         <axis xyz="0 1 0"/>
-        <limit effort="1000.0" velocity="1000.0"/>
-        <dynamics damping="1" friction="1"/>
+        <limit effort="1000" velocity="1000"/>
+        <dynamics damping="1.0" friction="1.0"/>
     </joint>
     <link name="wheel3_link">
         <visual>
-            <origin xyz="0 0 0" rpy="1.570795 0 0"/>
+            <origin xyz="0.0 0.0 0.0" rpy="1.570795 0 0"/>
             <geometry>
                 <cylinder radius="${wheel_link_radius}" length="${wheel_link_length}"/>
@@ -126,5 +128,5 @@
         </visual>
         <collision>
-            <origin xyz="0 0 0" rpy="1.570795 0 0"/>
+            <origin xyz="0.0 0.0 0.0" rpy="1.570795 0 0"/>
             <geometry>
                 <cylinder radius="${wheel_link_radius}" length="${wheel_link_length}"/>
@@ -138,13 +140,13 @@
         <parent link="body_link"/>
         <child link="wheel4_link"/>
-        <origin xyz="${body_link_x_dim/2 - wheel_link_radius/2} ${body_link_y_dim/2 + wheel_link_length/2} ${wheel_link_z_location}"
+        <origin xyz="${body_link_x_dim/2 - 1.2*wheel_link_radius} ${body_link_y_dim/2 + wheel_link_length/2} ${wheel_link_z_location}"
                 rpy="0.0 0.0 0.0"/>
         <axis xyz="0 1 0"/>
-        <limit effort="1000.0" velocity="1000"/>
-        <dynamics damping="1" friction="1"/>
+        <limit effort="1000" velocity="1000"/>
+        <dynamics damping="1.0" friction="1.0"/>
     </joint>
     <link name="wheel4_link">
         <visual>
-            <origin xyz="0 0 0" rpy="1.570795 0 0"/>
+            <origin xyz="0.0 0.0 0.0" rpy="1.570795 0 0"/>
             <geometry>
                 <cylinder radius="${wheel_link_radius}" length="${wheel_link_length}"/>
@@ -152,5 +154,5 @@
         </visual>
         <collision>
-            <origin xyz="0 0 0" rpy="1.570795 0 0"/>
+            <origin xyz="0.0 0.0 0.0" rpy="1.570795 0 0"/>
             <geometry>
                 <cylinder radius="${wheel_link_radius}" length="${wheel_link_length}"/>

File: urdf/car1.xacro (robot description, xacro)
@@ -19,5 +19,5 @@
         <inertial>
             <origin xyz="0.0 0.0 0.0" rpy="0.0 0.0 0.0"/>
-            <mass value="488"/>
+            <mass value="500"/>
             <inertia
                 ixx="0.014930555555555554"
@@ -36,12 +36,12 @@
     </link>
     <!-- Wheel template -->
-    <!-- wheel_mass = 1.7011193465, Izz = 0.00850559673, Ixx = Iyy = 0.00667468664 -->
+    <!-- wheel_mass = 22, Izz = 0.00850559673, Ixx = Iyy = 0.00667468664 -->
     <!-- Back right wheel -->
     <joint name="wheel1_joint" type="continuous">
         <parent link="body_link"/>
         <child link="wheel1_link"/>
-        <origin xyz="-0.45 -0.35 -0.1" rpy="0.0 0.0 0.0"/>
+        <origin xyz="-0.45 -0.35 -0.12" rpy="0.0 0.0 0.0"/>
         <axis xyz="0.0 1.0 0.0"/>
-        <limit effort="1000.0" velocity="1000.0"/>
+        <limit effort="1000.0" velocity="500"/>
         <dynamics damping="1" friction="1"/>
     </joint>
@@ -64,5 +64,5 @@
         <inertial>
             <origin rpy="0 0 0" xyz="0 0 0"/>
-            <mass value="1.7011193465"/>
+            <mass value="2"/>
             <inertia ixx="0.00667468664" ixy="0.0" ixz="0.0" iyy="0.00667468664" izz="0.00850559673" iyz="0"/>
         </inertial>
@@ -72,7 +72,7 @@
         <parent link="body_link"/>
         <child link="wheel2_link"/>
-        <origin xyz="-0.45 0.35 -0.1" rpy="0.0 0.0 0.0"/>
+        <origin xyz="-0.45 0.35 -0.12" rpy="0.0 0.0 0.0"/>
         <axis xyz="0 1 0"/>
-        <limit effort="1000.0" velocity="1000.0"/>
+        <limit effort="1000.0" velocity="500"/>
         <dynamics damping="1" friction="1"/>
     </joint>
@@ -92,5 +92,5 @@
         <inertial>
             <origin rpy="0 0 0" xyz="0 0 0"/>
-            <mass value="1.7011193465"/>
+            <mass value="2"/>
             <inertia ixx="0.00667468664" ixy="0.0" ixz="0.0" iyy="0.00667468664" izz="0.00850559673" iyz="0"/>
         </inertial>
@@ -100,7 +100,7 @@
         <parent link="body_link"/>
         <child link="wheel3_link"/>
-        <origin xyz="0.45 -0.35 -0.1" rpy="0.0 0.0 0.0"/>
+        <origin xyz="0.45 -0.35 -0.12" rpy="0.0 0.0 0.0"/>
         <axis xyz="0 1 0"/>
-        <limit effort="1000.0" velocity="1000.0"/>
+        <limit effort="1000.0" velocity="500"/>
         <dynamics damping="1" friction="1"/>
     </joint>
@@ -120,5 +120,5 @@
         <inertial>
             <origin rpy="0 0 0" xyz="0 0 0"/>
-            <mass value="1.7011193465"/>
+            <mass value="2"/>
             <inertia ixx="0.00667468664" ixy="0.0" ixz="0.0" iyy="0.00667468664" izz="0.00850559673" iyz="0"/>
         </inertial>
@@ -128,7 +128,7 @@
         <parent link="body_link"/>
         <child link="wheel4_link"/>
-        <origin xyz="0.45 0.35 -0.1" rpy="0.0 0.0 0.0"/>
+        <origin xyz="0.45 0.35 -0.12" rpy="0.0 0.0 0.0"/>
         <axis xyz="0 1 0"/>
-        <limit effort="1000.0" velocity="1000"/>
+        <limit effort="1000.0" velocity="500"/>
         <dynamics damping="1" friction="1"/>
     </joint>
@@ -148,7 +148,25 @@
         <inertial>
             <origin rpy="0 0 0" xyz="0 0 0"/>
-            <mass value="1.7011193465"/>
+            <mass value="2"/>
             <inertia ixx="0.00667468664" ixy="0.0" ixz="0.0" iyy="0.00667468664" izz="0.00850559673" iyz="0"/>
         </inertial>
     </link>
+    <!-- LiDAR sensor link -->
+    <joint name="lidar_joint" type="fixed">
+        <parent link="body_link"/>
+        <child link="lidar_link"/>
+        <!-- Gắn trên nóc xe, điều chỉnh cao độ và vị trí phù hợp -->
+        <origin xyz="0 0 0.2" rpy="0 0 0"/>
+    </joint>
+    <link name="lidar_link">
+    <visual>
+        <origin xyz="0 0 0" rpy="0 0 0"/>
+        <geometry>
+        <cylinder radius="0.05" length="0.02"/>
+        </geometry>
+        <material name="black">
+        <color rgba="0 0 0 1"/>
+        </material>
+    </visual>
+    </link>
 </robot>

Commit message: can use demo

File: urdf/car.xacro (robot description, xacro)
@@ -162,3 +162,37 @@
     </link>
     <!-- End front left wheel -->
+    <!-- Camera link -->
+    <joint name="camera_joint" type="fixed">
+        <parent link="body_link"/>
+        <child link="camera_link"/>
+        <origin xyz="0.2 0.0 0" rpy="0.0 0.0 0.0"/>
+    </joint>
+    <!-- Camera link with visual -->
+    <link name="camera_link">
+        <visual>
+            <origin xyz="0.0 0.0 0.2" rpy="0.0 0.0 0.0"/>
+            <geometry>
+                <!-- Here, we use a cylinder to represent the camera visually -->
+                <cylinder radius="0.05" length="0.1"/>
+            </geometry>
+        </visual>
+    </link>
+    <!-- End camera link -->
+    <!-- Front center sensor -->
+    <link name="front_sensor_link">
+        <visual>
+            <origin xyz="0 0 0.05" rpy="0 0 0"/>
+            <geometry>
+                <cylinder radius="0.05" length="0.1"/>
+            </geometry>
+            <material name="blue">
+                <color rgba="0 0 1 1"/>
+            </material>
+        </visual>
+    </link>
+    <joint name="front_sensor_joint" type="fixed">
+        <parent link="body_link"/>
+        <child link="front_sensor_link"/>
+        <origin xyz="0.5 0 0.1" rpy="0 0 0"/>
+    </joint>
 </robot>
